Commit message: next version of urdf - changed some positionings (added some other parts too, spinning wheels/lidar)

File: buddy_bot.urdf (robot description, URDF)
Before this commit: robot buddy_bot, 13 links, 12 joints
Links:
- link LIDAR: geometry collision cylinder length=.03 radius=.04; visual cylinder length=.03 radius=.04
- link back_wheel: geometry collision cylinder length=0.1 radius=0.095; visual cylinder length=0.1 radius=0.095
- link back_wheel_bar: geometry collision box size=.1 .1 .14; visual box size=.1 .1 .14
- link base_link: geometry collision box size=.6096 .4572 .3072; visual box size=.6096 .4572 .3072
- link front_connector: geometry collision box size=.03 .03 .4572; visual box size=.03 .03 .4572
- link front_left_bottom: geometry collision box size=.03 .03 .1677; visual box size=.03 .03 .1677
- link front_left_top: geometry collision box size=.03 .03 .35; visual box size=.03 .03 .35
- link front_right_bottom: geometry collision box size=.03 .03 .1677; visual box size=.03 .03 .1677
- link front_right_top: geometry collision box size=.03 .03 .35; visual box size=.03 .03 .35
- link front_wheel_bar: geometry collision box size=.1 .67 .14; visual box size=.1 .67 .14
- link left_wheel: geometry collision cylinder length=0.1 radius=0.095; visual cylinder length=0.1 radius=0.095
- link lidar_mount: geometry collision box size=.03 .03 .42; visual box size=.03 .03 .42
- link right_wheel: geometry collision cylinder length=0.1 radius=0.095; visual cylinder length=0.1 radius=0.095
