Commit message: buddybot loads into gazebo but it crashes

File: buddybot_ws/src/buddybot_description/urdf/buddybot.urdf (robot description, URDF)
Before this commit: robot buddy_bot, 13 links, 12 joints
Links:
- link LIDAR: mass None -> 1
- link back_wheel: mass None -> 1
- link back_wheel_bar: mass None -> 1
- link base_link: mass None -> 1
- link front_connector: mass None -> 1
- link front_left_bottom: mass None -> 1
- link front_left_top: mass None -> 1
- link front_right_bottom: mass None -> 1
- link front_right_top: mass None -> 1
- link front_wheel_bar: mass None -> 1
- link lidar_mount: mass None -> 1
- link right_wheel: mass None -> 1

Commit message: spawns buddybot without crashing

File: buddybot_ws/src/buddybot_description/urdf/buddybot.urdf (robot description, URDF)
Before this commit: robot buddy_bot, 13 links, 12 joints
Joints:
- joint bar_to_front_wheel_L: axis 0 1 0 -> (none); type continuous -> fixed
- joint bar_to_front_wheel_R: axis 0 1 0 -> (none); type continuous -> fixed
