Commit message: currently have navi spawn with hokuyo lidar

File: buddybot_ws/src/buddybot_description/urdf/buddybot.xacro (robot description, xacro)
@@ -1,4 +1,7 @@
 <?xml version="1.0"?>
-<robot name="buddy_bot">
+<!-- Revolute-Revolute Manipulator -->
+<robot name="buddybot" xmlns:xacro="http://www.ros.org/wiki/xacro">
+  <!-- Import all Gazebo-customization elements, including Gazebo colors -->
+  <xacro:include filename="$(find buddybot_description)/urdf/buddybot.gazebo" />
   <material name="blue">
     <color rgba="0 0 0.8 1"/>
@@ -66,5 +69,10 @@
         <cylinder length="0.1" radius="0.095"/>
       </geometry>
-    </collision>
+      <origin rpy="1.5708 0 0" xyz="0 0 0"/>
+    </collision>
+    <inertial>
+      <mass value="1"/>
+      <inertia ixx="1" ixy="0.0" ixz="0.0" iyy="1" iyz="0.0" izz="1"/>
+    </inertial>
   </link>
   <link name="right_wheel">
@@ -80,21 +88,44 @@
         <cylinder length="0.1" radius="0.095"/>
       </geometry>
-    </collision>
-    <inertial>
-      <mass value="1"/>
-      <inertia ixx="1" ixy="0.0" ixz="0.0" iyy="1" iyz="0.0" izz="1"/>
-    </inertial>
-  </link>
-  <joint name="bar_to_front_wheel_L" type="fixed">
+      <origin rpy="-1.6 0 0" xyz="0 0 0"/>
+    </collision>
+    <inertial>
+      <mass value="1"/>
+      <inertia ixx="1" ixy="0.0" ixz="0.0" iyy="1" iyz="0.0" izz="1"/>
+    </inertial>
+  </link>
+  <joint name="bar_to_front_wheel_L" type="continuous">
     <parent link="front_wheel_bar"/>
     <child link="left_wheel"/>
-    <!--<axis xyz="0 1 0"/>-->
+    <axis xyz="0 1 0"/>
     <origin xyz="0 0.34 -.08"/>
-  </joint>
-  <joint name="bar_to_front_wheel_R" type="fixed">
+    <dynamics damping="0.7"/>
+  </joint>
+  <transmission name="left_wheel_trans">
+    <type>transmission_interface/SimpleTransmission</type>
+    <joint name="bar_to_front_wheel_L">
+      <hardwareInterface>hardware_interface/EffortJointInterface</hardwareInterface>
+    </joint>
+    <actuator name="motor_left">
+      <hardwareInterface>hardware_interface/EffortJointInterface</hardwareInterface>
+      <mechanicalReduction>1</mechanicalReduction>
+    </actuator>
+  </transmission>
+  <transmission name="right_wheel_trans">
+    <type>transmission_interface/SimpleTransmission</type>
+    <joint name="bar_to_front_wheel_R">
+      <hardwareInterface>hardware_interface/EffortJointInterface</hardwareInterface>
+    </joint>
+    <actuator name="motor_right">
+      <hardwareInterface>hardware_interface/EffortJointInterface</hardwareInterface>
+      <mechanicalReduction>1</mechanicalReduction>
+    </actuator>
+  </transmission>
+  <joint name="bar_to_front_wheel_R" type="continuous">
     <parent link="front_wheel_bar"/>
     <child link="right_wheel"/>
-    <!--<axis xyz="0 1 0"/>-->
+    <axis xyz="0 1 0"/>
     <origin xyz="0 -0.34 -.08"/>
+    <dynamics damping="0.7"/>
   </joint>
   <link name = "back_wheel_bar">
@@ -133,4 +164,5 @@
         <cylinder length="0.1" radius="0.095"/>
       </geometry>
+      <origin rpy="-1.6 0 0" xyz="-0.1 0 0"/>
     </collision>
     <inertial>
@@ -144,4 +176,5 @@
     <axis xyz="0 0 1"/>
     <origin xyz="0 0 -.08"/>
+    <dynamics damping="0.7"/>
   </joint>
   <transmission name="back_wheel_turn">
@@ -177,25 +210,27 @@
     <origin xyz="-.3048 0 .50"/>
   </joint>
-  <link name = 'LIDAR'>
-    <visual>
-      <geometry>
-        <cylinder length = '.03' radius = '.04'/>
-      </geometry>
-      <origin rpy="0 0 0" xyz="0 0 0"/>
-      <material name= "black"/>
-    </visual>
-    <collision>
-      <geometry>
-        <cylinder length = '.03' radius = '.04'/>
-      </geometry>
-    </collision>
-    <inertial>
-      <mass value="1"/>
-      <inertia ixx="1" ixy="0.0" ixz="0.0" iyy="1" iyz="0.0" izz="1"/>
+ <!-- Hokuyo Laser -->
+  <link name="hokuyo_link">
+    <collision>
+      <origin xyz="0 0 0" rpy="0 0 0"/>
+      <geometry>
+	<box size="0.1 0.1 0.1"/>
+      </geometry>
+    </collision>
+    <visual>
+      <origin xyz="0 0 0" rpy="0 0 0"/>
+      <geometry>
+        <mesh filename="package://buddybot_description/meshes/hokuyo.dae"/>
+      </geometry>
+    </visual>
+    <inertial>
+      <mass value="1e-5" />
+      <origin xyz="0 0 0" rpy="0 0 0"/>
+      <inertia ixx="1e-6" ixy="0" ixz="0" iyy="1e-6" iyz="0" izz="1e-6" />
     </inertial>
   </link>
   <joint name = 'lidar_to_mount' type="fixed">
     <parent link="lidar_mount"/>
-    <child link="LIDAR"/>
+    <child link="hokuyo_link"/>
     <origin xyz="0 0 0"/>
   </joint>
@@ -315,10 +350,3 @@
     <origin xyz="0 0 0"/>
   </joint>
-   <!-- Gazebo plugin for ROS Control -->
-  <gazebo>
-    <plugin name="gazebo_ros_control" filename="libgazebo_ros_control.so">
-      <robotNamespace>/</robotNamespace>
-      <legacyModeNS>true</legacyModeNS>
-    </plugin>
-  </gazebo>
 </robot>

Commit message: got navi moving and with lidar

File: buddybot_ws/src/buddybot_description/urdf/buddybot.xacro (robot description, xacro)
@@ -17,4 +17,6 @@
   </material>
   <link name="base_link">
+  </link>
+  <link name="body">
     <visual>
       <geometry>
@@ -30,8 +32,13 @@
     </collision>
     <inertial>
-      <mass value="1"/>
-      <inertia ixx="1" ixy="0.0" ixz="0.0" iyy="1" iyz="0.0" izz="1"/>
-    </inertial>
-  </link>
+      <mass value="10"/>
+      <inertia ixx="1" ixy="0.0" ixz="0.0" iyy="1" iyz="0.0" izz="1"/>
+    </inertial>
+  </link>
+  <joint name = 'base_link_to_body' type = 'fixed'>
+    <parent link = 'base_link'/>
+    <child link = 'body'/>
+      <origin rpy="0 0 0" xyz="0 0 0"/>
+  </joint>
   <link name = "front_wheel_bar">
     <visual>
@@ -101,4 +108,5 @@
     <origin xyz="0 0.34 -.08"/>
     <dynamics damping="0.7"/>
+    <!--<pid p="100.0" i="0.0" d="10.0">-->
   </joint>
   <transmission name="left_wheel_trans">
@@ -128,4 +136,5 @@
     <origin xyz="0 -0.34 -.08"/>
     <dynamics damping="0.7"/>
+    <!--<pid p="100.0" i="0.0" d="10.0">-->
   </joint>
   <link name = "back_wheel_bar">
@@ -178,12 +187,13 @@
     <dynamics damping="0.7"/>
   </joint>
-  <transmission name="back_wheel_turn">
+  <transmission name="back_wheel_trans">
     <type>transmission_interface/SimpleTransmission</type>
-    <actuator name="$back_wheel_axis">
+    <joint name="back_bar_to_back_wheel">
+      <hardwareInterface>hardware_interface/EffortJointInterface</hardwareInterface>
+    </joint>
+    <actuator name="motor_back">
+      <hardwareInterface>hardware_interface/EffortJointInterface</hardwareInterface>
       <mechanicalReduction>1</mechanicalReduction>
     </actuator>
-    <joint name="back_bar_to_back_wheel">
-      <hardwareInterface>hardware_interface/PositionJointInterface</hardwareInterface>
-    </joint>
   </transmission>
   <link name = 'lidar_mount'>

Commit message: added kinect and moved lidar

File: buddybot_ws/src/buddybot_description/urdf/buddybot.xacro (robot description, xacro)
@@ -113,8 +113,8 @@
     <type>transmission_interface/SimpleTransmission</type>
     <joint name="bar_to_front_wheel_L">
-      <hardwareInterface>hardware_interface/EffortJointInterface</hardwareInterface>
+      <hardwareInterface>hardware_interface/VelocityJointInterface</hardwareInterface>
     </joint>
     <actuator name="motor_left">
-      <hardwareInterface>hardware_interface/EffortJointInterface</hardwareInterface>
+      <hardwareInterface>EffortJointInterface</hardwareInterface>
       <mechanicalReduction>1</mechanicalReduction>
     </actuator>
@@ -123,8 +123,8 @@
     <type>transmission_interface/SimpleTransmission</type>
     <joint name="bar_to_front_wheel_R">
-      <hardwareInterface>hardware_interface/EffortJointInterface</hardwareInterface>
+      <hardwareInterface>hardware_interface/VelocityJointInterface</hardwareInterface>
     </joint>
     <actuator name="motor_right">
-      <hardwareInterface>hardware_interface/EffortJointInterface</hardwareInterface>
+      <hardwareInterface>EffortJointInterface</hardwareInterface>
       <mechanicalReduction>1</mechanicalReduction>
     </actuator>
@@ -225,5 +225,5 @@
       <origin xyz="0 0 0" rpy="0 0 0"/>
       <geometry>
-	<box size="0.1 0.1 0.1"/>
+				<box size="0.1 0.1 0.1"/>
       </geometry>
     </collision>
@@ -240,99 +240,124 @@
     </inertial>
   </link>
+  <link name = 'front_right_top'>
+    <visual>
+      <geometry>
+        <box size = '.03 .03 .35'/>
+      </geometry>
+      <origin rpy="0 -.6 0" xyz=".4 0.215 0"/>
+      <material name = 'cyan'/>
+    </visual>
+    <collision>
+      <geometry>
+        <box size = '.03 .03 .35'/>
+      </geometry>
+    </collision>
+    <inertial>
+      <mass value="1"/>
+      <inertia ixx="1" ixy="0.0" ixz="0.0" iyy="1" iyz="0.0" izz="1"/>
+    </inertial>
+  </link>
+  <link name = 'front_left_top'>
+    <visual>
+      <geometry>
+        <box size = '.03 .03 .35'/>
+      </geometry>
+      <origin rpy="0 -.6 0" xyz=".4 -0.215 0"/>
+      <material name = 'cyan'/>
+    </visual>
+    <collision>
+      <geometry>
+        <box size = '.03 .03 .35'/>
+      </geometry>
+    </collision>
+    <inertial>
+      <mass value="1"/>
+      <inertia ixx="1" ixy="0.0" ixz="0.0" iyy="1" iyz="0.0" izz="1"/>
+    </inertial>
+  </link>
+  <link name = 'front_right_bottom'>
+    <visual>
+      <geometry>
+        <box size = '.03 .03 .1677'/>
+      </geometry>
+      <origin rpy="0 -1.6 0" xyz="0.42 .215 -.13"/>
+      <material name = 'cyan'/>
+    </visual>
+    <collision>
+      <geometry>
+        <box size = '.03 .03 .1677'/>
+      </geometry>
+    </collision>
+    <inertial>
+      <mass value="1"/>
+      <inertia ixx="1" ixy="0.0" ixz="0.0" iyy="1" iyz="0.0" izz="1"/>
+    </inertial>
+  </link>
+  <link name = 'front_left_bottom'>
+    <visual>
+      <geometry>
+        <box size = '.03 .03 .1677'/>
+      </geometry>
+      <origin rpy="0 -1.6 0" xyz="0.42 -.215 -.13"/>
+      <material name = 'cyan'/>
+    </visual>
+    <collision>
+      <geometry>
+        <box size = '.03 .03 .1677'/>
+      </geometry>
+    </collision>
+    <inertial>
+      <mass value="1"/>
+      <inertia ixx="1" ixy="0.0" ixz="0.0" iyy="1" iyz="0.0" izz="1"/>
+    </inertial>
+  </link>
+  <link name = 'front_connector'>
+    <visual>
+      <geometry>
+        <box size = '.03 .03 .4572'/>
+      </geometry>
+      <origin rpy="1.6 0 0" xyz=".5 0 -.13"/>
+      <material name = 'cyan'/>
+    </visual>
+    <collision>
+      <geometry>
+        <box size = '.03 .03 .4572'/>
+      </geometry>
+    </collision>
+    <inertial>
+      <mass value="1"/>
+      <inertia ixx="1" ixy="0.0" ixz="0.0" iyy="1" iyz="0.0" izz="1"/>
+    </inertial>
+  </link>
+  <!-- Realsense -->
+  <link name="realsense">
+    <collision>
+      <origin xyz="0 0 0" rpy="0 0 0"/>
+      <geometry>
+				<box size="0.073000 0.276000 0.072000"/>
+      </geometry>
+    </collision>
+    <visual>
+      <origin xyz="0 0 0" rpy="0 0 0"/>
+      <geometry>
+        <mesh filename="package://buddybot_description/meshes/kinect.dae"/>
+      </geometry>
+    </visual>
+    <inertial>
+      <mass value="0.1" />
+      <origin xyz="0 0 0" rpy="0 0 0"/>
+      <inertia ixx="9.108e-05" ixy="0.0" ixz="0.0" iyy="2.51e-06" iyz="0.0" izz="8.931e-05"/>
+		</inertial>
+  </link>
+  <joint name = 'camera_to_body' type="fixed">
+    <parent link="base_link"/>
+    <child link="hokuyo_link"/>
+    <origin xyz="0 0 .1886"/>
+  </joint>
   <joint name = 'lidar_to_mount' type="fixed">
     <parent link="lidar_mount"/>
-    <child link="hokuyo_link"/>
-    <origin xyz="0 0 0"/>
-  </joint>
-  <link name = 'front_right_top'>
-    <visual>
-      <geometry>
-        <box size = '.03 .03 .35'/>
-      </geometry>
-      <origin rpy="0 -.6 0" xyz=".4 0.215 0"/>
-      <material name = 'cyan'/>
-    </visual>
-    <collision>
-      <geometry>
-        <box size = '.03 .03 .35'/>
-      </geometry>
-    </collision>
-    <inertial>
-      <mass value="1"/>
-      <inertia ixx="1" ixy="0.0" ixz="0.0" iyy="1" iyz="0.0" izz="1"/>
-    </inertial>
-  </link>
-  <link name = 'front_left_top'>
-    <visual>
-      <geometry>
-        <box size = '.03 .03 .35'/>
-      </geometry>
-      <origin rpy="0 -.6 0" xyz=".4 -0.215 0"/>
-      <material name = 'cyan'/>
-    </visual>
-    <collision>
-      <geometry>
-        <box size = '.03 .03 .35'/>
-      </geometry>
-    </collision>
-    <inertial>
-      <mass value="1"/>
-      <inertia ixx="1" ixy="0.0" ixz="0.0" iyy="1" iyz="0.0" izz="1"/>
-    </inertial>
-  </link>
-  <link name = 'front_right_bottom'>
-    <visual>
-      <geometry>
-        <box size = '.03 .03 .1677'/>
-      </geometry>
-      <origin rpy="0 -1.6 0" xyz="0.42 .215 -.13"/>
-      <material name = 'cyan'/>
-    </visual>
-    <collision>
-      <geometry>
-        <box size = '.03 .03 .1677'/>
-      </geometry>
-    </collision>
-    <inertial>
-      <mass value="1"/>
-      <inertia ixx="1" ixy="0.0" ixz="0.0" iyy="1" iyz="0.0" izz="1"/>
-    </inertial>
-  </link>
-  <link name = 'front_left_bottom'>
-    <visual>
-      <geometry>
-        <box size = '.03 .03 .1677'/>
-      </geometry>
-      <origin rpy="0 -1.6 0" xyz="0.42 -.215 -.13"/>
-      <material name = 'cyan'/>
-    </visual>
-    <collision>
-      <geometry>
-        <box size = '.03 .03 .1677'/>
-      </geometry>
-    </collision>
-    <inertial>
-      <mass value="1"/>
-      <inertia ixx="1" ixy="0.0" ixz="0.0" iyy="1" iyz="0.0" izz="1"/>
-    </inertial>
-  </link>
-  <link name = 'front_connector'>
-    <visual>
-      <geometry>
-        <box size = '.03 .03 .4572'/>
-      </geometry>
-      <origin rpy="1.6 0 0" xyz=".5 0 -.13"/>
-      <material name = 'cyan'/>
-    </visual>
-    <collision>
-      <geometry>
-        <box size = '.03 .03 .4572'/>
-      </geometry>
-    </collision>
-    <inertial>
-      <mass value="1"/>
-      <inertia ixx="1" ixy="0.0" ixz="0.0" iyy="1" iyz="0.0" izz="1"/>
-    </inertial>
-  </link>
+    <child link="realsense"/>
+    <origin xyz=".04 0 .032"/>
+  </joint>
   <joint name = 'F_R_T_to_base' type = 'fixed'>
     <parent link="base_link"/>

Commit message: edit inertia

File: buddybot_ws/src/buddybot_description/urdf/buddybot.xacro (robot description, xacro)
@@ -33,5 +33,5 @@
     <inertial>
       <mass value="10"/>
-      <inertia ixx="1" ixy="0.0" ixz="0.0" iyy="1" iyz="0.0" izz="1"/>
+      <inertia ixx="0.38832" ixy="0.0" ixz="0.0" iyy="0.48387" iyz="0.0" izz="0.25283"/>
     </inertial>
   </link>
@@ -56,5 +56,5 @@
     <inertial>
       <mass value="1"/>
-      <inertia ixx="1" ixy="0.0" ixz="0.0" iyy="1" iyz="0.0" izz="1"/>
+      <inertia ixx="0.002466" ixy="0.0" ixz="0.0" iyy="0.038241" iyz="0.0" izz="0.039041"/>
     </inertial>
   </link>
@@ -153,5 +153,5 @@
     <inertial>
       <mass value="1"/>
-      <inertia ixx="1" ixy="0.0" ixz="0.0" iyy="1" iyz="0.0" izz="1"/>
+      <inertia ixx="0.002466" ixy="0.0" ixz="0.0" iyy="0.001666" iyz="0.0" izz="0.002466"/>
     </inertial>
   </link>
@@ -212,5 +212,5 @@
     <inertial>
       <mass value="1"/>
-      <inertia ixx="1" ixy="0.0" ixz="0.0" iyy="1" iyz="0.0" izz="1"/>
+      <inertia ixx="0.01477" ixy="0.0" ixz="0.0" iyy="0.00015" iyz="0.0" izz="0.01477"/>
     </inertial>
   </link>
@@ -255,5 +255,5 @@
     <inertial>
       <mass value="1"/>
-      <inertia ixx="1" ixy="0.0" ixz="0.0" iyy="1" iyz="0.0" izz="1"/>
+      <inertia ixx="0.01028" ixy="0.0" ixz="0.0" iyy="0.00015" iyz="0.0" izz="0.01028"/>
     </inertial>
   </link>
@@ -273,5 +273,5 @@
     <inertial>
       <mass value="1"/>
-      <inertia ixx="1" ixy="0.0" ixz="0.0" iyy="1" iyz="0.0" izz="1"/>
+      <inertia ixx="0.01028" ixy="0.0" ixz="0.0" iyy="0.00015" iyz="0.0" izz="0.01028"/>
     </inertial>
   </link>

Commit message: added moments for boxes

File: buddybot_ws/src/buddybot_description/urdf/buddybot.xacro (robot description, xacro)
@@ -291,5 +291,5 @@
     <inertial>
       <mass value="1"/>
-      <inertia ixx="1" ixy="0.0" ixz="0.0" iyy="1" iyz="0.0" izz="1"/>
+      <inertia ixx="0.002419" ixy="0.0" ixz="0.0" iyy="0.00015" iyz="0.0" izz="0.002419"/>
     </inertial>
   </link>
@@ -309,5 +309,5 @@
     <inertial>
       <mass value="1"/>
-      <inertia ixx="1" ixy="0.0" ixz="0.0" iyy="1" iyz="0.0" izz="1"/>
+      <inertia ixx="0.002419" ixy="0.0" ixz="0.0" iyy="0.00015" iyz="0.0" izz="0.002419"/>
     </inertial>
   </link>
@@ -327,5 +327,5 @@
     <inertial>
       <mass value="1"/>
-      <inertia ixx="1" ixy="0.0" ixz="0.0" iyy="1" iyz="0.0" izz="1"/>
+      <inertia ixx="0.01749" ixy="0.0" ixz="0.0" iyy="0.00015" iyz="0.0" izz="0.01749"/>
     </inertial>
   </link>

Commit message: finished dimentions/moments of all links

File: buddybot_ws/src/buddybot_description/urdf/buddybot.xacro (robot description, xacro)
@@ -79,6 +79,6 @@
     </collision>
     <inertial>
-      <mass value="1"/>
-      <inertia ixx="1" ixy="0.0" ixz="0.0" iyy="1" iyz="0.0" izz="1"/>
+      <mass value="3"/>
+      <inertia ixx="0.0092687" ixy="0.0" ixz="0.0" iyy="0.0092687" iyz="0.0" izz="0.0022563"/>
     </inertial>
   </link>
@@ -98,6 +98,6 @@
     </collision>
     <inertial>
-      <mass value="1"/>
-      <inertia ixx="1" ixy="0.0" ixz="0.0" iyy="1" iyz="0.0" izz="1"/>
+      <mass value="3"/>
+      <inertia ixx="0.0092687" ixy="0.0" ixz="0.0" iyy="0.0092687" iyz="0.0" izz="0.0022563"/>
     </inertial>
   </link>
@@ -176,6 +176,6 @@
     </collision>
     <inertial>
-      <mass value="1"/>
-      <inertia ixx="1" ixy="0.0" ixz="0.0" iyy="1" iyz="0.0" izz="1"/>
+      <mass value="3"/>
+      <inertia ixx="0.0092687" ixy="0.0" ixz="0.0" iyy="0.0092687" iyz="0.0" izz="0.0022563"/>
     </inertial>
   </link>

Commit message: modified back wheel to rotate on two axes

File: buddybot_ws/src/buddybot_description/urdf/buddybot.xacro (robot description, xacro)
@@ -159,17 +159,42 @@
     <origin xyz = '-.28 0 -.2'/>
   </joint>
+  <link name="back_wheel_roller">
+    <visual>
+      <geometry>
+        <cylinder length="0.005" radius="0.005"/>
+      </geometry>
+      <origin rpy="-1.6 0 0" xyz="-0 .12 .12"/>
+      <material name="cyan"/>
+    </visual>
+    <collision>
+      <geometry>
+        <cylinder length="0.1" radius="0.005"/>
+      </geometry>
+      <origin rpy="-1.6 0 0" xyz="-0 0 0"/>
+    </collision>
+    <inertial>
+      <mass value="1"/>
+      <inertia ixx="0.0001458" ixy="0.0" ixz="0.0" iyy="0.0001458" iyz="0.0" izz="0.00001458"/>
+    </inertial>
+  </link>
+  <joint name="back_bar_to_back_wheel_roller" type="continuous">
+    <parent link="back_wheel_bar"/>
+    <child link="back_wheel_roller"/>
+    <axis xyz="0 0 1"/>
+    <origin xyz="-0.15 0 -.07"/>
+  </joint>
   <link name="back_wheel">
     <visual>
       <geometry>
-        <cylinder length="0.1" radius="0.095"/>
-      </geometry>
-      <origin rpy="-1.6 0 0" xyz="-0.1 0 0"/>
+        <cylinder length="0.06" radius="0.095"/>
+      </geometry>
+      <origin rpy="-1.6 0 0" xyz="-0 0 0"/>
       <material name="black"/>
     </visual>
     <collision>
       <geometry>
-        <cylinder length="0.1" radius="0.095"/>
-      </geometry>
-      <origin rpy="-1.6 0 0" xyz="-0.1 0 0"/>
+        <cylinder length="0.06" radius="0.095"/>
+      </geometry>
+      <origin rpy="-1.6 0 0" xyz="-0 0 0"/>
     </collision>
     <inertial>
@@ -178,9 +203,9 @@
     </inertial>
   </link>
-  <joint name="back_bar_to_back_wheel" type="continuous">
-    <parent link="back_wheel_bar"/>
+  <joint name="back_wheel_roller_to_back_wheel" type="continuous">
+    <parent link="back_wheel_roller"/>
     <child link="back_wheel"/>
-    <axis xyz="0 0 1"/>
-    <origin xyz="0 0 -.08"/>
+    <axis xyz="0 1 0"/>
+    <origin xyz="0 0 0"/>
   </joint>
  <!-- Hokuyo Laser -->

Commit message: modified back wheel to rotate on two axes

File: buddybot_ws/src/buddybot_description/urdf/buddybot.xacro (robot description, xacro)
@@ -214,5 +214,5 @@
       <origin xyz="0 0 0" rpy="0 0 0"/>
       <geometry>
-	<box size="0.1 0.1 0.1"/>
+  <box size="0.1 0.1 0.1"/>
       </geometry>
     </collision>

Commit message: fixed back wheel to work like a roller wheel

File: buddybot_ws/src/buddybot_description/urdf/buddybot.xacro (robot description, xacro)
@@ -154,32 +154,14 @@
     </inertial>
   </link>
-  <joint name = 'base_to_back_wheel_bar' type = 'fixed'>
+  <joint name = 'base_to_back_wheel_bar' type = 'continuous'>
     <parent link = 'body'/>
     <child link = 'back_wheel_bar'/>
+    <axis xyz="0 0 1"/>
     <origin xyz = '-.28 0 -.2'/>
   </joint>
-  <link name="back_wheel_roller">
-    <visual>
-      <geometry>
-        <cylinder length="0.005" radius="0.005"/>
-      </geometry>
-      <origin rpy="-1.6 0 0" xyz="-0 .12 .12"/>
-      <material name="cyan"/>
-    </visual>
-    <collision>
-      <geometry>
-        <cylinder length="0.1" radius="0.005"/>
-      </geometry>
-      <origin rpy="-1.6 0 0" xyz="-0 0 0"/>
-    </collision>
-    <inertial>
-      <mass value="1"/>
-      <inertia ixx="0.0001458" ixy="0.0" ixz="0.0" iyy="0.0001458" iyz="0.0" izz="0.00001458"/>
-    </inertial>
-  </link>
-  <joint name="back_bar_to_back_wheel_roller" type="continuous">
+  <joint name="back_bar_to_back_wheel" type="continuous">
     <parent link="back_wheel_bar"/>
-    <child link="back_wheel_roller"/>
-    <axis xyz="0 0 1"/>
+    <child link="back_wheel"/>
+    <axis xyz="0 1 0"/>
     <origin xyz="-0.15 0 -.07"/>
   </joint>
@@ -203,10 +185,4 @@
     </inertial>
   </link>
-  <joint name="back_wheel_roller_to_back_wheel" type="continuous">
-    <parent link="back_wheel_roller"/>
-    <child link="back_wheel"/>
-    <axis xyz="0 1 0"/>
-    <origin xyz="0 0 0"/>
-  </joint>
  <!-- Hokuyo Laser -->
   <link name="hokuyo_link">

Commit message: resource added

File: buddybot_ws/src/buddybot_description/urdf/buddybot.xacro (robot description, xacro)
@@ -186,5 +186,5 @@
   </link>
  <!-- Hokuyo Laser -->
-  <link name="hokuyo_link">
+  <link name="laser">
     <collision>
       <origin xyz="0 0 0" rpy="0 0 0"/>
@@ -207,5 +207,5 @@
   <joint name = 'lidar_to_body' type="fixed">
     <parent link="body"/>
-    <child link="hokuyo_link"/>
+    <child link="laser"/>
     <origin xyz="0 0 .1886"/>
   </joint>
